File: Electronics/Appendix/4700/ALU/cmos_inv.kicad_sch (KiCad schematic)
At the start: 4 parts, among them T1 NMOS, T1'1 PMOS, X1 Conn_01x01_Socket

Commit message: fixing cmos_inf
Parts:
- removed OUT2: (no value), symbol Connector:Conn_01x01_Socket
- removed X1: Conn_01x01_Socket, symbol Connector:Conn_01x01_Socket
- renumbered T1'1 to T1, T1 to T2
Connections:
- net INV_OUT: now reaches T1.1 (D), T2.1 (D)
- net INV_IN: now reaches T1.2 (G), T2.2 (G)
Changed lines of the file:
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@@
 		)
 	)
-	(symbol
-		(lib_id "Connector:Conn_01x01_Socket")
-		(at 158.75 76.2 0)
-		(unit 1)
-		(body_style 1)
-		(exclude_from_sim no)
-		(in_bom yes)
-		(on_board yes)
-		(in_pos_files yes)
-		(dnp no)
-		(fields_autoplaced yes)
-		(property "Reference" "OUT2"
-			(at 160.02 74.9299 0)
-			(show_name no)
-			(do_not_autoplace no)
-			(effects
-				(font
-					(size 1.27 1.27)
-				)
-				(justify left)
-			)
-		)
-		(property "Value" ""
-			(at 160.02 77.4699 0)
-			(show_name no)
-			(do_not_autoplace no)
-			(effects
-				(font
-					(size 1.27 1.27)
-				)
-				(justify left)
-			)
-		)
-		(property "Footprint" ""
-			(at 158.75 76.2 0)
-			(hide yes)
-			(show_name no)
-			(do_not_autoplace no)
-			(effects
-				(font
-					(size 1.27 1.27)
-				)
-			)
-		)
-		(property "Datasheet" ""
-			(at 158.75 76.2 0)
-			(hide yes)
-			(show_name no)
-			(do_not_autoplace no)
-			(effects
-				(font
-					(size 1.27 1.27)
-				)
-			)
-		)
-		(property "Description" "Generic connector, single row, 01x01, script generated"
-			(at 158.75 76.2 0)
-			(hide yes)
-			(show_name no)
-			(do_not_autoplace no)
-			(effects
-				(font
-					(size 1.27 1.27)
-				)
-			)
-		)
-		(pin "1"
-		)
-		(instances
-			(project "Test"
-				(path "/0a7a9431-a390-42ce-aae4-32a0355adbaa"
-					(reference "OUT1")
-					(unit 1)
-				)
-			)
-			(project "cmos_inv"
-				(path "/6cce6f8f-6df3-4cbb-becc-12ed677d66be"
-					(reference "OUT1")
-					(unit 1)
-				)
-			)
-			(project "cmos_xnor2"
-				(path "/fd146099-cfa7-464c-817b-4439fed62346/cc31ddaf-13b5-42b1-ab3e-d1a54ede226c"
-					(reference "OUT2")
-					(unit 1)
-				)
-			)
+	(hierarchical_label "INV_OUT"
+		(shape input)
+		(at 153.67 76.2 0)
+		(effects
+			(font
+				(size 1.27 1.27)
+			)
+			(justify left)
+		)
+	)
+	(hierarchical_label "INV_IN"
+		(shape input)
+		(at 123.19 76.2 180)
+		(effects
+			(font
+				(size 1.27 1.27)
+			)
+			(justify right)
 		)
 	)
@@
 	)
 	(symbol
-		(lib_id "Connector:Conn_01x01_Socket")
-		(at 118.11 76.2 0)
-		(mirror y)
-		(unit 1)
-		(body_style 1)
-		(exclude_from_sim no)
-		(in_bom yes)
-		(on_board yes)
-		(in_pos_files yes)
-		(dnp no)
-		(property "Reference" "X1"
-			(at 116.84 74.9299 0)
-			(show_name no)
-			(do_not_autoplace no)
-			(effects
-				(font
-					(size 1.27 1.27)
-				)
-				(justify left)
-			)
-		)
-		(property "Value" "Conn_01x01_Socket"
-			(at 116.84 77.4699 0)
-			(hide yes)
-			(show_name no)
-			(do_not_autoplace no)
-			(effects
-				(font
-					(size 1.27 1.27)
-				)
-				(justify left)
-			)
-		)
-		(property "Footprint" ""
-			(at 118.11 76.2 0)
-			(hide yes)
-			(show_name no)
-			(do_not_autoplace no)
-			(effects
-				(font
-					(size 1.27 1.27)
-				)
-			)
-		)
-		(property "Datasheet" ""
-			(at 118.11 76.2 0)
-			(hide yes)
-			(show_name no)
-			(do_not_autoplace no)
-			(effects
-				(font
-					(size 1.27 1.27)
-				)
-			)
-		)
-		(property "Description" "Generic connector, single row, 01x01, script generated"
-			(at 118.11 76.2 0)
-			(hide yes)
-			(show_name no)
-			(do_not_autoplace no)
-			(effects
-				(font
-					(size 1.27 1.27)
-				)
-			)
-		)
-		(pin "1"
-		)
-		(instances
-			(project "Test"
-				(path "/0a7a9431-a390-42ce-aae4-32a0355adbaa"
-					(reference "X1")
-					(unit 1)
-				)
-			)
-			(project "cmos_inv"
-				(path "/6cce6f8f-6df3-4cbb-becc-12ed677d66be"
-					(reference "X1")
-					(unit 1)
-				)
-			)
-			(project "cmos_xnor2"
-				(path "/fd146099-cfa7-464c-817b-4439fed62346/cc31ddaf-13b5-42b1-ab3e-d1a54ede226c"
-					(reference "X1")
-					(unit 1)
-				)
-			)
-		)
-	)
-	(symbol
 		(lib_id "power:GND")
 		(at 140.97 93.98 0)
@@
 		(dnp no)
 		(fields_autoplaced yes)
-		(property "Reference" "T1"
+		(property "Reference" "T2"
 			(at 144.78 83.8199 0)
 			(show_name no)
@@
 		(in_pos_files yes)
 		(dnp no)
-		(property "Reference" "T1'1"
+		(property "Reference" "T1"
 			(at 145.034 65.786 0)
 			(show_name no)
@@
 		)
 	)
+	(sheet_instances
+		(path "/"
+			(page "1")
+		)
+	)
+	(embedded_fonts no)
 )
